Commit message: sv aSd

File: cr5_moveit/config/cr5_robot.xacro.urdf (robot description, URDF)
Before this commit: robot cr5_robot, 11 links, 10 joints
Links:
- added link camera_link, mass 0.05; collision box size=0.03 0.03 0.02; visual box size=0.03 0.03 0.02
- link camera_color_optical_frame: mass 0.05 -> None; geometry 
Joints:
- added joint camera_color_optiacl_frame_joint: type fixed, parent camera_link, child camera_color_optical_frame, origin xyz=0 0 0 rpy=-1.57 0 -1.57
- joint wrist_camera_fixed: child camera_color_optical_frame -> camera_link; origin xyz=0.05 0.005 0.03 rpy=0 0 0 -> xyz=0.05 0.005 0.03 rpy=1.57 -1.57 0
